File: 27c160-adaptor/27c160.sch (KiCad schematic (older format))
At the start: 6 parts, among them P1 A19_SEL, P2 A18_SEL, U1 27C4096, U2 27C160

Commit message: made a THT version for easier soldering
Parts:
- P1, P2: symbol CONN_01X03 -> Jumper:Jumper_3_Open
- R1, R2: footprint Resistors_SMD:R_0805_HandSoldering -> Resistor_THT:R_Axial_DIN0207_L6.3mm_D2.5mm_P7.62mm_Horizontal; symbol R -> Device:R
- U1: symbol MAPLE_MINI -> FF:MAPLE_MINI
- U2: symbol MAPLE_MINI_48 -> FF:MAPLE_MINI_48
Connections:
- wire segments 92 -> 94
Changed lines of the file:
@@
-EESchema Schematic File Version 2
-LIBS:power
-LIBS:device
-LIBS:transistors
-LIBS:conn
-LIBS:linear
-LIBS:regul
-LIBS:74xx
-LIBS:cmos4000
-LIBS:adc-dac
-LIBS:memory
-LIBS:xilinx
-LIBS:microcontrollers
-LIBS:dsp
-LIBS:microchip
-LIBS:analog_switches
-LIBS:motorola
-LIBS:texas
-LIBS:intel
-LIBS:audio
-LIBS:interface
-LIBS:digital-audio
-LIBS:philips
-LIBS:display
-LIBS:cypress
-LIBS:siliconi
-LIBS:opto
-LIBS:atmel
-LIBS:contrib
-LIBS:valves
-LIBS:FF
-LIBS:27c160-cache
-EELAYER 25 0
+EESchema Schematic File Version 4
+EELAYER 30 0
 EELAYER END
 $Descr A4 11693 8268
@@
 $EndDescr
 $Comp
-L MAPLE_MINI U1
+L FF:MAPLE_MINI U1
 U 1 1 55AF4EC7
 P 3550 2200
@@
 $EndComp
 $Comp
-L MAPLE_MINI_48 U2
+L FF:MAPLE_MINI_48 U2
 U 1 1 55AF4F2A
 P 7000 2200
@@
 A19
 $Comp
-L CONN_01X03 P2
+L Jumper:Jumper_3_Open P2
 U 1 1 55F952CF
-P 7450 1300
-F 0 "P2" H 7450 1500 50  0000 C CNN
-F 1 "A18_SEL" V 7550 1300 50  0000 C CNN
-F 2 "Pin_Headers:Pin_Header_Straight_1x03" H 7450 1300 60  0001 C CNN
-F 3 "" H 7450 1300 60  0000 C CNN
-	1    7450 1300
-	1    0    0    -1
-$EndComp
-$Comp
-L CONN_01X03 P1
+P 7250 1300
+F 0 "P2" H 7250 1500 50  0000 C CNN
+F 1 "A18_SEL" V 7350 1300 50  0000 C CNN
+F 2 "Pin_Headers:Pin_Header_Straight_1x03" H 7250 1300 60  0001 C CNN
+F 3 "~" H 7250 1300 60  0000 C CNN
+	1    7250 1300
+	0    1    1    0
+$EndComp
+$Comp
+L Jumper:Jumper_3_Open P1
 U 1 1 55F953E8
-P 6700 1300
-F 0 "P1" H 6700 1500 50  0000 C CNN
-F 1 "A19_SEL" V 6800 1300 50  0000 C CNN
-F 2 "Pin_Headers:Pin_Header_Straight_1x03" H 6700 1300 60  0001 C CNN
-F 3 "" H 6700 1300 60  0000 C CNN
-	1    6700 1300
-	1    0    0    -1
-$EndComp
-$Comp
-L R R2
+P 6500 1300
+F 0 "P1" H 6500 1500 50  0000 C CNN
+F 1 "A19_SEL" V 6600 1300 50  0000 C CNN
+F 2 "Pin_Headers:Pin_Header_Straight_1x03" H 6500 1300 60  0001 C CNN
+F 3 "~" H 6500 1300 60  0000 C CNN
+	1    6500 1300
+	0    1    1    0
+$EndComp
+$Comp
+L Device:R R2
 U 1 1 55F954A1
 P 6150 1600
 F 0 "R2" V 6230 1600 50  0000 C CNN
 F 1 "1K" V 6150 1600 50  0000 C CNN
-F 2 "Resistors_SMD:R_0805_HandSoldering" V 6080 1600 30  0001 C CNN
+F 2 "Resistor_THT:R_Axial_DIN0207_L6.3mm_D2.5mm_P7.62mm_Horizontal" V 6080 1600 30  0001 C CNN
 F 3 "" H 6150 1600 30  0000 C CNN
 	1    6150 1600
@@
 $EndComp
 $Comp
-L R R1
+L Device:R R1
 U 1 1 55F954FE
 P 6150 900
 F 0 "R1" V 6230 900 50  0000 C CNN
 F 1 "1K" V 6150 900 50  0000 C CNN
-F 2 "Resistors_SMD:R_0805_HandSoldering" V 6080 900 30  0001 C CNN
+F 2 "Resistor_THT:R_Axial_DIN0207_L6.3mm_D2.5mm_P7.62mm_Horizontal" V 6080 900 30  0001 C CNN
 F 3 "" H 6150 900 30  0000 C CNN
 	1    6150 900
@@
 VSS
 Wire Wire Line
-	6300 1600 7250 1600
-Wire Wire Line
-	7250 1600 7250 1400
-Wire Wire Line
-	6500 1400 6500 1600
+	6300 1600 6500 1600
+Wire Wire Line
+	7250 1600 7250 1550
+Wire Wire Line
+	6500 1550 6500 1600
 Connection ~ 6500 1600
 Wire Wire Line
-	6300 900  7250 900
-Wire Wire Line
-	7250 900  7250 1200
-Wire Wire Line
-	6500 1200 6500 900
+	6300 900  6500 900
+Wire Wire Line
+	7250 900  7250 1050
+Wire Wire Line
+	6500 1050 6500 900
 Connection ~ 6500 900
 Wire Wire Line
-	6500 1300 6300 1300
-Wire Wire Line
-	7250 1300 7050 1300
-Text Label 7050 1300 0    60   ~ 0
+	6350 1300 6150 1300
+Wire Wire Line
+	7100 1300 6900 1300
+Text Label 6950 1300 0    60   ~ 0
 A18
-Text Label 6300 1300 0    60   ~ 0
+Text Label 6200 1300 0    60   ~ 0
 A19
+Wire Wire Line
+	6500 1600 7250 1600
+Wire Wire Line
+	6500 900  7250 900
 $EndSCHEMATC
