File: greaseweazle/GW.sch (KiCad schematic (older format))
At the start: 8 parts, among them P5 POWER, P7 FLOPPY, U1 TAOBAO

Commit message: made a THT version for easier soldering
Parts:
- R1, R2, R3, R4, R5: footprint Resistors_SMD:R_0805_HandSoldering -> Resistor_THT:R_Axial_DIN0207_L6.3mm_D2.5mm_P7.62mm_Horizontal
Changed lines of the file:
@@
 EESchema Schematic File Version 4
-LIBS:GW-cache
-EELAYER 26 0
+EELAYER 30 0
 EELAYER END
 $Descr A4 11693 8268
@@
 F 0 "R2" V 9330 4100 50  0000 C CNN
 F 1 "1K" V 9250 4100 50  0000 C CNN
-F 2 "Resistors_SMD:R_0805_HandSoldering" V 9180 4100 30  0001 C CNN
+F 2 "Resistor_THT:R_Axial_DIN0207_L6.3mm_D2.5mm_P7.62mm_Horizontal" V 9180 4100 30  0001 C CNN
 F 3 "" H 9250 4100 30  0000 C CNN
 	1    9250 4100
@@
 F 0 "R3" V 9480 4100 50  0000 C CNN
 F 1 "1K" V 9400 4100 50  0000 C CNN
-F 2 "Resistors_SMD:R_0805_HandSoldering" V 9330 4100 30  0001 C CNN
+F 2 "Resistor_THT:R_Axial_DIN0207_L6.3mm_D2.5mm_P7.62mm_Horizontal" V 9330 4100 30  0001 C CNN
 F 3 "" H 9400 4100 30  0000 C CNN
 	1    9400 4100
@@
 F 0 "R4" V 9630 4100 50  0000 C CNN
 F 1 "1K" V 9550 4100 50  0000 C CNN
-F 2 "Resistors_SMD:R_0805_HandSoldering" V 9480 4100 30  0001 C CNN
+F 2 "Resistor_THT:R_Axial_DIN0207_L6.3mm_D2.5mm_P7.62mm_Horizontal" V 9480 4100 30  0001 C CNN
 F 3 "" H 9550 4100 30  0000 C CNN
 	1    9550 4100
@@
 F 0 "R5" V 9780 4100 50  0000 C CNN
 F 1 "1K" V 9700 4100 50  0000 C CNN
-F 2 "Resistors_SMD:R_0805_HandSoldering" V 9630 4100 30  0001 C CNN
+F 2 "Resistor_THT:R_Axial_DIN0207_L6.3mm_D2.5mm_P7.62mm_Horizontal" V 9630 4100 30  0001 C CNN
 F 3 "" H 9700 4100 30  0000 C CNN
 	1    9700 4100
@@
 F 0 "R1" V 5880 6150 50  0000 C CNN
 F 1 "1.5K" V 5800 6150 50  0000 C CNN
-F 2 "Resistors_SMD:R_0805_HandSoldering" V 5730 6150 30  0001 C CNN
+F 2 "Resistor_THT:R_Axial_DIN0207_L6.3mm_D2.5mm_P7.62mm_Horizontal" V 5730 6150 30  0001 C CNN
 F 3 "" H 5800 6150 30  0000 C CNN
 	1    5800 6150
