File: greaseweazle/GW.kicad_pcb (KiCad board)
At the start: 2 copper layers, 61 x 22.9 mm, 8 parts, among them P5 POWER, P7 FLOPPY, U1 TAOBAO

Commit message: added SilkScreen for resistors on back side added "usbpu" to resistor R1
Parts:
- R1 USBPU: renamed from R1
Other:
- board text added: "PC Drive Rev 1a"
- board text added: "R1 USBPU"
- board text added: "R2"
- board text added: "R3"
- board text added: "R4"
- board text added: "R5"
- board text removed: "PC Drive Rev 1"
Changed lines of the file:
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@@
   (general
     (thickness 1.6)
-    (drawings 11)
+    (drawings 16)
     (tracks 115)
     (zones 0)
@@
       (effects (font (size 1 1) (thickness 0.15)) (justify mirror))
     )
-    (fp_text value FLOPPY (at -2.03186 -18.9809 180) (layer B.SilkS)
+    (fp_text value FLOPPY (at 4.83884 -34.132 180) (layer B.SilkS)
       (effects (font (size 1 1) (thickness 0.15)) (justify mirror))
     )
@@
     (descr "Resistor, Axial_DIN0207 series, Axial, Horizontal, pin pitch=7.62mm, 0.25W = 1/4W, length*diameter=6.3*2.5mm^2, http://cdn-reichelt.de/documents/datenblatt/B400/1_4W%23YAG.pdf")
     (tags "Resistor Axial_DIN0207 series Axial Horizontal pin pitch 7.62mm 0.25W = 1/4W length 6.3mm diameter 2.5mm")
-    (fp_text reference R1 (at 3.8608 -2.032) (layer F.SilkS)
+    (fp_text reference "R1 USBPU" (at 3.8608 -2.032) (layer F.SilkS)
       (effects (font (size 1 1) (thickness 0.15)))
     )
@@
     )
   )
+  (gr_text R2 (at 168.402 108.712) (layer B.SilkS)
+    (effects (font (size 1 1) (thickness 0.15)) (justify mirror))
+  )
+  (gr_text R5 (at 160.528 108.712) (layer B.SilkS)
+    (effects (font (size 1 1) (thickness 0.15)) (justify mirror))
+  )
+  (gr_text R4 (at 130.302 108.712) (layer B.SilkS)
+    (effects (font (size 1 1) (thickness 0.15)) (justify mirror))
+  )
+  (gr_text R3 (at 140.335 108.712) (layer B.SilkS)
+    (effects (font (size 1 1) (thickness 0.15)) (justify mirror))
+  )
+  (gr_text "R1 USBPU" (at 150.495 108.712) (layer B.SilkS)
+    (effects (font (size 1 1) (thickness 0.15)) (justify mirror))
+  )
   (gr_text JLCJLCJLCJLC (at 149.2504 100.9396) (layer F.SilkS)
     (effects (font (size 1.5 1.5) (thickness 0.3)))
@@
     (effects (font (size 1.5 1.5) (thickness 0.3)))
   )
-  (gr_text "PC Drive Rev 1" (at 138.43 100.965) (layer B.SilkS)
+  (gr_text "PC Drive Rev 1a" (at 136.779 99.949) (layer B.SilkS)
     (effects (font (size 1.5 1.5) (thickness 0.3)) (justify mirror))
   )
@@
     (effects (font (size 1 1) (thickness 0.15)) (justify mirror))
   )
-  (gr_text Greaseweazle (at 171.45 100.965) (layer B.SilkS)
+  (gr_text Greaseweazle (at 171.704 100.711) (layer B.SilkS)
     (effects (font (size 2.2 2.2) (thickness 0.45)) (justify left mirror))
   )
